Commit message: add sensors

File: urdf/ackermann_robot.urdf (robot description, URDF)
Before this commit: robot ackermann_robot, 14 links, 13 joints
Links:
- added link cam1; collision box size=0.02 0.02 0.02; visual box size=0.02 0.02 0.02
- added link cam1_undis; collision box size=0.028 0.028 0.028; visual box size=0.028 0.028 0.028
Joints:
- added joint cam1_joint: type fixed, parent cam0, child cam1, origin xyz=0 -0.0936 0 rpy=0 0 0
- added joint cam1_undis_joint: type fixed, parent cam1, child cam1_undis, origin xyz=0 0 0 rpy=-1.5707963268 0 -1.5707963268

Commit message: update 2D viewer mannual in readme

File: urdf/ackermann_robot.urdf (robot description, URDF)
Before this commit: robot ackermann_robot, 16 links, 15 joints
Joints:
- joint cam0_joint: origin xyz=0 0 0.058 rpy=0 0 0 -> xyz=0 0.0936 0.058 rpy=0 0 0
